File: TrashFlash/TrashFlash.kicad_pcb (KiCad board)
At the start: 2 copper layers, 105 x 45 mm, 113 parts, among them IC1 LTC3643IUDD#PBF, IC10 BQ24230RGTR, IC11 STM32L471QEI6, IC2 ADG5419BCPZ-RL7, IC3 BQ27426YZFR, IC4 SN74LXC2T45QDTTRQ1, IC5 TPS63900DSKR, IC6 TPS63900DSKR, IC7 LP5024RSMR, IC8 AD8615AUJZ-REEL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

Commit message: Old changes
Parts:
- added BT1: 628, TrashFlash:BAT_628, F.Cu at (57.4, 88.0)
- added BT2: 5223, TrashFlash:BAT_5223, F.Cu at (101.0, 89.0)
- added LED1: 150353M153300, TrashFlash:150353M153300, F.Cu at (105.0, 95.0)
Connections:
- LED2 pad 2: /User_Interface/RED0 -> /User_Interface/RED2
- LED2 pad 4: /User_Interface/GREEN0 -> /User_Interface/GREEN2
- LED2 pad 6: /User_Interface/BLUE0 -> /User_Interface/BLUE2
- LED3 pad 2: /User_Interface/RED0 -> /User_Interface/RED1
- LED3 pad 4: /User_Interface/GREEN0 -> /User_Interface/GREEN1
- LED3 pad 6: /User_Interface/BLUE0 -> /User_Interface/BLUE1
- LED4 pad 2: /User_Interface/RED0 -> /User_Interface/RED3
- LED4 pad 4: /User_Interface/GREEN0 -> /User_Interface/GREEN3
- LED4 pad 6: /User_Interface/BLUE0 -> /User_Interface/BLUE3
- LED5 pad 2: /User_Interface/RED0 -> /User_Interface/RED4
- LED5 pad 4: /User_Interface/GREEN0 -> /User_Interface/GREEN4
- LED5 pad 6: /User_Interface/BLUE0 -> /User_Interface/BLUE4
- LED6 pad 2: /User_Interface/RED0 -> /User_Interface/RED5
- LED6 pad 4: /User_Interface/GREEN0 -> /User_Interface/GREEN5
- LED6 pad 6: /User_Interface/BLUE0 -> /User_Interface/BLUE5
- LED7 pad 2: /User_Interface/RED0 -> /User_Interface/RED6
- LED7 pad 4: /User_Interface/GREEN0 -> /User_Interface/GREEN6
- LED7 pad 6: /User_Interface/BLUE0 -> /User_Interface/BLUE6
- LED8 pad 2: /User_Interface/RED0 -> /User_Interface/RED7
- LED8 pad 4: /User_Interface/GREEN0 -> /User_Interface/GREEN7
- LED8 pad 6: /User_Interface/BLUE0 -> /User_Interface/BLUE7
