File: TrashFlash/LED_Supply.kicad_sch (KiCad schematic)
At the start: 14 parts, among them IC1 LTC3643IUDD#PBF

Commit message: Added Wireless and inter PCB connector
Parts:
- added C304, C305: 10u, Capacitor_SMD:C_1206_3216Metric, symbol Device:C
- C303: renamed from C7; value 22u -> 10u; footprint Capacitor_SMD:C_0603_1608Metric -> Capacitor_SMD:C_1206_3216Metric
- IC301: renamed from IC1; footprint TrashFlash:QFN50P300X500X80-25N-D -> QFN50P300X500X80-25N-D
- L301: renamed from L1; footprint TrashFlash:INDPM5454X310N -> INDPM5454X310N
- renumbered C5 to C301, C6 to C302, C8 to C306, C9 to C307, C10 to C308, C11 to C309, R10 to R301, R14 to R302, R17 to R303, R15 to R304, R16 to R305
Connections:
- net GND: now also C304.2, C305.2
- net Vdrive: now also C304.1, C305.1
Other:
- moved on the sheet: C306

Commit message: Added battery and connectors, Schematic remark for BQ297xx
Parts:
- IC301: footprint QFN50P300X500X80-25N-D -> TrashFlash:QFN50P300X500X80-25N-D
- L301: footprint INDPM5454X310N -> TrashFlash:INDPM5454X310N
Changed lines of the file:
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@@
 			)
 		)
-		(property "Footprint" "QFN50P300X500X80-25N-D"
+		(property "Footprint" "TrashFlash:QFN50P300X500X80-25N-D"
 			(at 127.254 172.974 0)
 			(effects
@@
 			)
 		)
-		(property "Footprint" "INDPM5454X310N"
+		(property "Footprint" "TrashFlash:INDPM5454X310N"
 			(at 187.96 131.75 0)
 			(effects
@@
 			)
 		)
-		(property "Footprint" "QFN50P300X500X80-25N-D"
+		(property "Footprint" "TrashFlash:QFN50P300X500X80-25N-D"
 			(at 127.254 82.804 0)
 			(effects
