File: TrashFlash/Supply.kicad_sch (KiCad schematic)
At the start: 13 parts, among them IC501 TPS63900DSKR, IC502 TPS63900DSKR

Commit message: Added battery and connectors, Schematic remark for BQ297xx
Parts:
- IC501, IC502: footprint SON50P250X250X80-11N-D -> TrashFlash:SON50P250X250X80-11N-D
- L501, L502: footprint INDM2016X100N -> TrashFlash:INDM2016X100N
Changed lines of the file:
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@@
 			)
 		)
-		(property "Footprint" "INDM2016X100N"
+		(property "Footprint" "TrashFlash:INDM2016X100N"
 			(at 162.56 193.98 0)
 			(effects
@@
 			)
 		)
-		(property "Footprint" "SON50P250X250X80-11N-D"
+		(property "Footprint" "TrashFlash:SON50P250X250X80-11N-D"
 			(at 162.56 131.75 0)
 			(effects
@@
 			)
 		)
-		(property "Footprint" "SON50P250X250X80-11N-D"
+		(property "Footprint" "TrashFlash:SON50P250X250X80-11N-D"
 			(at 162.56 201.6 0)
 			(effects
@@
 			)
 		)
-		(property "Footprint" "INDM2016X100N"
+		(property "Footprint" "TrashFlash:INDM2016X100N"
 			(at 162.56 124.13 0)
 			(effects
