File: TrashFlash/Wireless_Interface.kicad_sch (KiCad schematic)
At the start: 29 parts, among them IC801 CC110LRGPR, Y801 ECS-260-10-33B-CKM-TR

Commit message: Moved USB and added JTAG connector
Parts:
- L801, L802, L803, L804, L805, L806, L807: footprint Inductor_SMD:L_01005_0402Metric -> Inductor_SMD:L_0402_1005Metric
Changed lines of the file:
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@@
 			)
 		)
-		(property "Footprint" "Inductor_SMD:L_01005_0402Metric"
+		(property "Footprint" "Inductor_SMD:L_0402_1005Metric"
 			(at 196.85 48.26 0)
 			(effects
@@
 			)
 		)
-		(property "Footprint" "Inductor_SMD:L_01005_0402Metric"
+		(property "Footprint" "Inductor_SMD:L_0402_1005Metric"
 			(at 209.55 48.26 0)
 			(effects
@@
 			)
 		)
-		(property "Footprint" "Inductor_SMD:L_01005_0402Metric"
+		(property "Footprint" "Inductor_SMD:L_0402_1005Metric"
 			(at 171.45 41.91 0)
 			(effects
@@
 			)
 		)
-		(property "Footprint" "Inductor_SMD:L_01005_0402Metric"
+		(property "Footprint" "Inductor_SMD:L_0402_1005Metric"
 			(at 184.15 41.91 0)
 			(effects
@@
 			)
 		)
-		(property "Footprint" "Inductor_SMD:L_01005_0402Metric"
+		(property "Footprint" "Inductor_SMD:L_0402_1005Metric"
 			(at 177.8 60.96 0)
 			(effects
@@
 			)
 		)
-		(property "Footprint" "Inductor_SMD:L_01005_0402Metric"
+		(property "Footprint" "Inductor_SMD:L_0402_1005Metric"
 			(at 171.45 54.61 0)
 			(effects
@@
 			)
 		)
-		(property "Footprint" "Inductor_SMD:L_01005_0402Metric"
+		(property "Footprint" "Inductor_SMD:L_0402_1005Metric"
 			(at 246.38 48.26 0)
 			(effects

Commit message: Added battery and connectors, Schematic remark for BQ297xx
Parts:
- ANT801: footprint ANTC7020X90N -> TrashFlash:ANTC7020X90N
- IC801: footprint QFN50P400X400X100-21N-D -> TrashFlash:QFN50P400X400X100-21N-D
- Y801: footprint ECS160833B2CTNTR3 -> TrashFlash:ECS160833B2CTNTR3
Changed lines of the file:
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@@
 			)
 		)
-		(property "Footprint" "ECS160833B2CTNTR3"
+		(property "Footprint" "TrashFlash:ECS160833B2CTNTR3"
 			(at 146.05 93.98 0)
 			(effects
@@
 			)
 		)
-		(property "Footprint" "ANTC7020X90N"
+		(property "Footprint" "TrashFlash:ANTC7020X90N"
 			(at 289.56 145.72 0)
 			(effects
@@
 			)
 		)
-		(property "Footprint" "QFN50P400X400X100-21N-D"
+		(property "Footprint" "TrashFlash:QFN50P400X400X100-21N-D"
 			(at 81.28 126.238 0)
 			(effects
